Commit message: Added m-explore-ros2 content directly

File: install/vac_bot/share/vac_bot/description/robot_core.xacro (robot description, xacro)
@@ -14,24 +14,16 @@
         <color rgba="0 0 0 1"/>
     </material>
+        <!-- BASE FOOTPRINT -->]
+    <link name="base_footprint"></link>
+    <joint name="base_footprint_joint" type="fixed">
+        <parent link="base_footprint"/>
+        <child link="base_link"/>
+        <origin xyz="0 0 0" rpy="0 0 0"/>
+    </joint>
     <!-- BASE LINK -->
     <link name="base_link">
-    </link>
-    <!-- BASE FOOTPRINT -->
-    <joint name="base_footprint_joint" type="fixed">
-        <parent link="base_link"/>
-        <child link="base_footprint"/>
-        <origin xyz="0 0 0" rpy="0 0 0"/>
-    </joint>
-    <link name="base_footprint">
-    </link>
-    <!-- CHASSIS LINK -->
-    <joint name="chassis_joint" type="fixed">
-        <parent link="base_link"/>
-        <child link="chassis"/>
-        <origin xyz="-0.1 0 0"/>
-    </joint>
-    <link name="chassis">
+    <pose>0 0 0.1 0 0 0</pose>
         <visual>
-            <origin xyz="0.15 0 0.0325"/>
+            <origin xyz="0 0 0.0325"/>
             <geometry>
                 <cylinder radius="0.2" length="0.1"/>
@@ -40,5 +32,5 @@
         </visual>
         <collision>
-            <origin xyz="0.15 0 0.0325"/>
+            <origin xyz="0 0 0.0325"/>
             <geometry>
                 <cylinder radius="0.2" length="0.1"/>
@@ -46,6 +38,32 @@
         </collision>
         <xacro:inertial_cylinder mass="0.5" length="0.1" radius="0.2">
-            <origin xyz="0.15 0 0.0325" rpy="0 0 0"/>
+            <origin xyz="0 0 0.0325" rpy="0 0 0"/>
         </xacro:inertial_cylinder>
+        <visual name="front_caster_wheel_visual">
+            <origin xyz="0.15 0 -0.0025" rpy="0 0 0"/>
+            <geometry>
+                <sphere radius="0.03"/>
+            </geometry>
+            <material name="black"/>
+        </visual>
+        <collision name="front_caster_wheel_collision">
+            <origin xyz="0.15 0 -0.0025" rpy="0 0 0"/>
+            <geometry>
+                <sphere radius="0.03"/>
+            </geometry>
+        </collision>
+        <visual name="rear_caster_wheel_visual">
+            <origin xyz="-0.15 0 -0.0025" rpy="0 0 0"/>
+            <geometry>
+                <sphere radius="0.03"/>
+            </geometry>
+            <material name="black"/>
+        </visual>
+        <collision name="rear_caster_wheel_collision">
+            <origin xyz="-0.15 0 -0.0025" rpy="0 0 0"/>
+            <geometry>
+                <sphere radius="0.03"/>
+            </geometry>
+        </collision>
     </link>
     <!-- LEFT WHEEL LINK -->
@@ -55,4 +73,6 @@
         <origin xyz="0.05 0.09 0" rpy="-${pi/2} 0 0" />
         <axis xyz="0 0 1"/>
+        <limit effort="100" velocity="20.0"/>
+        <dynamics damping="2.0" friction="3.0"/>
     </joint>
     <link name="left_wheel">
@@ -78,4 +98,6 @@
         <origin xyz="0.05 -0.09 0" rpy="${pi/2} 0 0" />
         <axis xyz="0 0 -1"/>
+        <limit effort="100" velocity="20.0"/>
+        <dynamics damping="2.0" friction="3.0"/>
     </joint>
     <link name="right_wheel">
@@ -95,30 +117,3 @@
         </xacro:inertial_cylinder>
     </link>
-    <!-- CASTER WHEEL LINK -->
-    <joint name="caster_wheel_joint" type="fixed">
-        <parent link="chassis"/>
-        <child link="caster_wheel"/>
-        <origin xyz="0.3 0 -0.0025"/>
-    </joint>
-    <link name="caster_wheel">
-        <visual>
-            <geometry>
-                <sphere radius="0.03"/>
-            </geometry>
-            <material name="black"/>
-        </visual>
-        <collision>
-            <geometry>
-                <sphere radius="0.03"/>
-            </geometry>
-        </collision>
-        <xacro:inertial_sphere mass="0.1" radius="0.03">
-            <origin xyz="0 0 0" rpy="0 0 0"/>
-        </xacro:inertial_sphere>
-    </link>
-    <gazebo reference="caster_wheel">
-        <material>Gazebo/White</material>
-        <mu1 value="0.001"/>
-        <mu2 value="0.001"/>
-    </gazebo>
 </robot>

File: vac_bot/src/vac_bot/description/robot_core.xacro (robot description, xacro)
@@ -14,24 +14,15 @@
         <color rgba="0 0 0 1"/>
     </material>
+        <!-- BASE FOOTPRINT -->]
+    <link name="base_footprint"></link>
+    <joint name="base_footprint_joint" type="fixed">
+        <parent link="base_footprint"/>
+        <child link="base_link"/>
+        <origin xyz="0 0 0" rpy="0 0 0"/>
+    </joint>
     <!-- BASE LINK -->
     <link name="base_link">
-    </link>
-    <!-- BASE FOOTPRINT -->
-    <joint name="base_footprint_joint" type="fixed">
-        <parent link="base_link"/>
-        <child link="base_footprint"/>
-        <origin xyz="0 0 0" rpy="0 0 0"/>
-    </joint>
-    <link name="base_footprint">
-    </link>
-    <!-- CHASSIS LINK -->
-    <joint name="chassis_joint" type="fixed">
-        <parent link="base_link"/>
-        <child link="chassis"/>
-        <origin xyz="-0.1 0 0"/>
-    </joint>
-    <link name="chassis">
         <visual>
-            <origin xyz="0.15 0 0.0325"/>
+            <origin xyz="0 0 0.0325"/>
             <geometry>
                 <cylinder radius="0.2" length="0.1"/>
@@ -40,5 +31,5 @@
         </visual>
         <collision>
-            <origin xyz="0.15 0 0.0325"/>
+            <origin xyz="0 0 0.0325"/>
             <geometry>
                 <cylinder radius="0.2" length="0.1"/>
@@ -46,6 +37,32 @@
         </collision>
         <xacro:inertial_cylinder mass="0.5" length="0.1" radius="0.2">
-            <origin xyz="0.15 0 0.0325" rpy="0 0 0"/>
+            <origin xyz="0 0 0.0325" rpy="0 0 0"/>
         </xacro:inertial_cylinder>
+        <visual name="front_caster_wheel_visual">
+            <origin xyz="0.15 0 -0.0025" rpy="0 0 0"/>
+            <geometry>
+                <sphere radius="0.03"/>
+            </geometry>
+            <material name="black"/>
+        </visual>
+        <collision name="front_caster_wheel_collision">
+            <origin xyz="0.15 0 -0.0025" rpy="0 0 0"/>
+            <geometry>
+                <sphere radius="0.03"/>
+            </geometry>
+        </collision>
+        <visual name="rear_caster_wheel_visual">
+            <origin xyz="-0.15 0 -0.0025" rpy="0 0 0"/>
+            <geometry>
+                <sphere radius="0.03"/>
+            </geometry>
+            <material name="black"/>
+        </visual>
+        <collision name="rear_caster_wheel_collision">
+            <origin xyz="-0.15 0 -0.0025" rpy="0 0 0"/>
+            <geometry>
+                <sphere radius="0.03"/>
+            </geometry>
+        </collision>
     </link>
     <!-- LEFT WHEEL LINK -->
@@ -55,4 +72,6 @@
         <origin xyz="0.05 0.09 0" rpy="-${pi/2} 0 0" />
         <axis xyz="0 0 1"/>
+        <limit effort="100" velocity="20.0"/>
+        <dynamics damping="2.0" friction="3.0"/>
     </joint>
     <link name="left_wheel">
@@ -78,4 +97,6 @@
         <origin xyz="0.05 -0.09 0" rpy="${pi/2} 0 0" />
         <axis xyz="0 0 -1"/>
+        <limit effort="100" velocity="20.0"/>
+        <dynamics damping="2.0" friction="3.0"/>
     </joint>
     <link name="right_wheel">
@@ -95,30 +116,3 @@
         </xacro:inertial_cylinder>
     </link>
-    <!-- CASTER WHEEL LINK -->
-    <joint name="caster_wheel_joint" type="fixed">
-        <parent link="chassis"/>
-        <child link="caster_wheel"/>
-        <origin xyz="0.3 0 -0.0025"/>
-    </joint>
-    <link name="caster_wheel">
-        <visual>
-            <geometry>
-                <sphere radius="0.03"/>
-            </geometry>
-            <material name="black"/>
-        </visual>
-        <collision>
-            <geometry>
-                <sphere radius="0.03"/>
-            </geometry>
-        </collision>
-        <xacro:inertial_sphere mass="0.1" radius="0.03">
-            <origin xyz="0 0 0" rpy="0 0 0"/>
-        </xacro:inertial_sphere>
-    </link>
-    <gazebo reference="caster_wheel">
-        <material>Gazebo/White</material>
-        <mu1 value="0.001"/>
-        <mu2 value="0.001"/>
-    </gazebo>
 </robot>
