Commit message: fixed velocity, next make the URDF back to normal

File: install/vac_bot/share/vac_bot/description/gazebo_control.xacro (robot description, xacro)
@@ -3,14 +3,19 @@
    <gazebo>
         <plugin name="gz::sim::systems::DiffDrive" filename="gz-sim-diff-drive-system">
-            <!-- Wheel Information -->
             <left_joint>left_wheel_joint</left_joint>
             <right_joint>right_wheel_joint</right_joint>
             <wheel_separation>0.18</wheel_separation>
             <wheel_radius>0.0325</wheel_radius>
-            <!-- <max_wheel_torque>200</max_wheel_torque> -->
-            <max_linear_acceleration>0.33</max_linear_acceleration>
-            <!-- Limits -->
+            <!-- Control gains and limits (optional) -->
+            <max_velocity>3.0</max_velocity>                <!-- Max linear velocity in m/s -->
+            <max_linear_acceleration>1</max_linear_acceleration>
+            <min_linear_acceleration>-1</min_linear_acceleration>
+            <max_angular_acceleration>2</max_angular_acceleration>
+            <min_angular_acceleration>-2</min_angular_acceleration>
+            <max_linear_velocity>0.5</max_linear_velocity>
+            <min_linear_velocity>-0.5</min_linear_velocity>
+            <max_angular_velocity>1</max_angular_velocity>
+            <min_angular_velocity>-1</min_angular_velocity>
             <topic>cmd_vel</topic>
-            <!-- Output -->
             <frame_id>odom</frame_id>
             <child_frame_id>base_link</child_frame_id>

File: install/vac_bot/share/vac_bot/description/lidar.xacro (robot description, xacro)
@@ -2,7 +2,7 @@
 <robot xmlns:xacro="http://www.ros.org/wiki/xacro" >
     <joint name="laser_joint" type="fixed">
-        <parent link="chassis"/>
+        <parent link="base_link"/>
         <child link="laser_frame"/>
-        <origin xyz="0.24 0 0.09" rpy="0 0 0"/>
+        <origin xyz="0.09 0 0.09" rpy="0 0 0"/>
     </joint>
     <link name="laser_frame">

File: install/vac_bot/share/vac_bot/description/robot_core.xacro (robot description, xacro)
@@ -23,6 +23,15 @@
     <!-- BASE LINK -->
     <link name="base_link">
-    <pose>0 0 0.1 0 0 0</pose>
-        <visual>
+        <pose>0 0 0.1 0 0 0</pose>
+        <xacro:inertial_cylinder mass="1.5" length="0.1" radius="0.2">
+            <origin xyz="0.0 0 0.0325" rpy="0 0 0"/>
+        </xacro:inertial_cylinder>
+        <collision name="base_link_collision">
+            <origin xyz="0 0 0.0325"/>
+            <geometry>
+                <cylinder radius="0.2" length="0.1"/>
+            </geometry>
+        </collision>
+        <visual name="base_link_visual">
             <origin xyz="0 0 0.0325"/>
             <geometry>
@@ -31,13 +40,10 @@
             <material name="white"/>
         </visual>
-        <collision>
-            <origin xyz="0 0 0.0325"/>
+        <collision name="front_caster_wheel_collision">
+            <origin xyz="0.15 0 -0.0025" rpy="0 0 0"/>
             <geometry>
-                <cylinder radius="0.2" length="0.1"/>
+                <sphere radius="0.03"/>
             </geometry>
         </collision>
-        <xacro:inertial_cylinder mass="0.5" length="0.1" radius="0.2">
-            <origin xyz="0 0 0.0325" rpy="0 0 0"/>
-        </xacro:inertial_cylinder>
         <visual name="front_caster_wheel_visual">
             <origin xyz="0.15 0 -0.0025" rpy="0 0 0"/>
@@ -47,6 +53,6 @@
             <material name="black"/>
         </visual>
-        <collision name="front_caster_wheel_collision">
-            <origin xyz="0.15 0 -0.0025" rpy="0 0 0"/>
+        <collision name="rear_caster_wheel_collision">
+            <origin xyz="-0.15 0 -0.0025" rpy="0 0 0"/>
             <geometry>
                 <sphere radius="0.03"/>
@@ -60,10 +66,4 @@
             <material name="black"/>
         </visual>
-        <collision name="rear_caster_wheel_collision">
-            <origin xyz="-0.15 0 -0.0025" rpy="0 0 0"/>
-            <geometry>
-                <sphere radius="0.03"/>
-            </geometry>
-        </collision>
     </link>
     <!-- LEFT WHEEL LINK -->
@@ -71,8 +71,8 @@
         <parent link="base_link"/>
         <child link="left_wheel"/>
-        <origin xyz="0.05 0.09 0" rpy="-${pi/2} 0 0" />
+        <origin xyz="0 0.09 0" rpy="-${pi/2} 0 0" />
         <axis xyz="0 0 1"/>
-        <limit effort="100" velocity="20.0"/>
-        <dynamics damping="2.0" friction="3.0"/>
+        <limit effort="100" velocity="10.0"/>
+        <dynamics damping="1.0" friction="1.0"/>
     </joint>
     <link name="left_wheel">
@@ -96,8 +96,8 @@
         <parent link="base_link"/>
         <child link="right_wheel"/>
-        <origin xyz="0.05 -0.09 0" rpy="${pi/2} 0 0" />
+        <origin xyz="0 -0.09 0" rpy="${pi/2} 0 0" />
         <axis xyz="0 0 -1"/>
-        <limit effort="100" velocity="20.0"/>
-        <dynamics damping="2.0" friction="3.0"/>
+        <limit effort="100" velocity="10.0"/>
+        <dynamics damping="1.0" friction="1.0"/>
     </joint>
     <link name="right_wheel">

File: vac_bot/src/vac_bot/description/robot_core.xacro (robot description, xacro)
@@ -23,5 +23,15 @@
     <!-- BASE LINK -->
     <link name="base_link">
-        <visual>
+        <pose>0 0 0.1 0 0 0</pose>
+        <xacro:inertial_cylinder mass="1.5" length="0.1" radius="0.2">
+            <origin xyz="0.0 0 0.0325" rpy="0 0 0"/>
+        </xacro:inertial_cylinder>
+        <collision name="base_link_collision">
+            <origin xyz="0 0 0.0325"/>
+            <geometry>
+                <cylinder radius="0.2" length="0.1"/>
+            </geometry>
+        </collision>
+        <visual name="base_link_visual">
             <origin xyz="0 0 0.0325"/>
             <geometry>
@@ -30,13 +40,10 @@
             <material name="white"/>
         </visual>
-        <collision>
-            <origin xyz="0 0 0.0325"/>
+        <collision name="front_caster_wheel_collision">
+            <origin xyz="0.15 0 -0.0025" rpy="0 0 0"/>
             <geometry>
-                <cylinder radius="0.2" length="0.1"/>
+                <sphere radius="0.03"/>
             </geometry>
         </collision>
-        <xacro:inertial_cylinder mass="0.5" length="0.1" radius="0.2">
-            <origin xyz="0 0 0.0325" rpy="0 0 0"/>
-        </xacro:inertial_cylinder>
         <visual name="front_caster_wheel_visual">
             <origin xyz="0.15 0 -0.0025" rpy="0 0 0"/>
@@ -46,6 +53,6 @@
             <material name="black"/>
         </visual>
-        <collision name="front_caster_wheel_collision">
-            <origin xyz="0.15 0 -0.0025" rpy="0 0 0"/>
+        <collision name="rear_caster_wheel_collision">
+            <origin xyz="-0.15 0 -0.0025" rpy="0 0 0"/>
             <geometry>
                 <sphere radius="0.03"/>
@@ -59,10 +66,4 @@
             <material name="black"/>
         </visual>
-        <collision name="rear_caster_wheel_collision">
-            <origin xyz="-0.15 0 -0.0025" rpy="0 0 0"/>
-            <geometry>
-                <sphere radius="0.03"/>
-            </geometry>
-        </collision>
     </link>
     <!-- LEFT WHEEL LINK -->
@@ -70,8 +71,8 @@
         <parent link="base_link"/>
         <child link="left_wheel"/>
-        <origin xyz="0.05 0.09 0" rpy="-${pi/2} 0 0" />
+        <origin xyz="0 0.09 0" rpy="-${pi/2} 0 0" />
         <axis xyz="0 0 1"/>
-        <limit effort="100" velocity="20.0"/>
-        <dynamics damping="2.0" friction="3.0"/>
+        <limit effort="100" velocity="10.0"/>
+        <dynamics damping="1.0" friction="1.0"/>
     </joint>
     <link name="left_wheel">
@@ -95,8 +96,8 @@
         <parent link="base_link"/>
         <child link="right_wheel"/>
-        <origin xyz="0.05 -0.09 0" rpy="${pi/2} 0 0" />
+        <origin xyz="0 -0.09 0" rpy="${pi/2} 0 0" />
         <axis xyz="0 0 -1"/>
-        <limit effort="100" velocity="20.0"/>
-        <dynamics damping="2.0" friction="3.0"/>
+        <limit effort="100" velocity="10.0"/>
+        <dynamics damping="1.0" friction="1.0"/>
     </joint>
     <link name="right_wheel">
