Commit message: add slam toolbox

File: vac_bot/src/vac_bot/description/robot_core.xacro (robot description, xacro)
@@ -16,4 +16,12 @@
     <!-- BASE LINK -->
     <link name="base_link">
+    </link>
+    <!-- BASE FOOTPRINT -->
+    <joint name="base_footprint_joint" type="fixed">
+        <parent link="base_link"/>
+        <child link="base_footprint"/>
+        <origin xyz="0 0 0" rpy="0 0 0"/>
+    </joint>
+    <link name="base_footprint">
     </link>
     <!-- CHASSIS LINK -->
